File: 40s-2040rmie.kicad_sch (KiCad schematic)
At the start: 195 parts, among them U1 RP2040, U2 SRV05-4, U3 W25Q128JVS, U4 XC6206PxxxMR, Y1 12MHz

Commit message: commit work from months ago, forget what i did
Parts:
- removed D1, D60, D61, D62: D_Small, Diode_SMD:D_SOD-123, symbol Device:D_Small
- removed MX0-0, MX1-B12, MX4-0_0, MX4-10_2, MX4-1_2, MX4-4_3, MX4-7_2, MX4-7_3: MX-NoLED, marbastlib-mx:SW_MX_1u, symbol MX_Alps_Hybrid:MX-NoLED
- removed MX4-0_1, MX4-11_1, MX4-2_1, MX4-9_1: MX-NoLED, marbastlib-mx:SW_MX_1.5u, symbol MX_Alps_Hybrid:MX-NoLED
- removed MX4-11_2, MX4-2_2, MX4-3_4, MX4-8_4, MX4-9_2: MX-NoLED, marbastlib-mx:SW_MX_1.25u, symbol MX_Alps_Hybrid:MX-NoLED
- removed MX4-4_4, MX4-7_4: MX-NoLED, marbastlib-mx:SW_MX_1.75u, symbol MX_Alps_Hybrid:MX-NoLED
- removed ST-1_0: 10u (8u), marbastlib-mx:STAB_MX_10u, symbol marbastlib-mx:MX_stab
- removed ST-2_0: 6u, marbastlib-mx:STAB_MX_6u, symbol marbastlib-mx:MX_stab
- removed ST-3_0, ST-3_1: 3u, marbastlib-mx:STAB_MX_3u, symbol marbastlib-mx:MX_stab
- removed ST-A_0: 2u, marbastlib-mx:STAB_MX_2u, symbol marbastlib-mx:MX_stab
- MX0-1, MX0-10, MX0-11, MX0-12, MX0-13, MX0-14, MX0-15, MX0-2, MX0-3, MX0-4, MX0-5, MX0-6, MX0-9, MX1-0, MX1-1, MX1-10, MX1-11, MX1-13, MX1-14, MX1-15, MX1-2, MX1-3, MX1-4, MX1-5, MX1-6, MX1-7, MX1-8, MX1-9, MX2-1, MX2-10, MX2-2, MX2-3, MX2-4, MX2-5, MX2-6, MX2-7, MX2-8, MX2-9, MX3-1, MX3-10, MX3-14, MX3-2, MX3-3, MX3-4, MX3-5, MX3-6, MX3-7, MX3-8, MX3-9, MX4-13, MX4-14, MX4-15: footprint marbastlib-mx:SW_MX_1u -> Valve:SW_MX_1u
- MX1-12: renamed from MX1-A12; footprint marbastlib-mx:SW_MX_1u -> Valve:SW_MX_1u
- MX2-0, MX3-11: footprint marbastlib-mx:SW_MX_1.25u -> Valve:SW_MX_1.25u
- MX2-11, MX3-0: footprint marbastlib-mx:SW_MX_1.75u -> Valve:SW_MX_1.75u
- MX4-0: renamed from MX4-0_2; footprint marbastlib-mx:SW_MX_1.25u -> Valve:SW_MX_1.25u
- MX4-1: renamed from MX4-1_0; footprint marbastlib-mx:SW_MX_1u -> Valve:SW_MX_1.25u
- MX4-10: renamed from MX4-10_0; footprint marbastlib-mx:SW_MX_1u -> Valve:SW_MX_1u
- MX4-11: renamed from MX4-11_0; footprint marbastlib-mx:SW_MX_1u -> Valve:SW_MX_1u
- MX4-2: renamed from MX4-2_0; footprint marbastlib-mx:SW_MX_1u -> Valve:SW_MX_1.25u
- MX4-5: renamed from MX4-4_0; footprint marbastlib-mx:SW_MX_1u -> Valve:SW_MX_1u
- MX4-9: renamed from MX4-9_0; footprint marbastlib-mx:SW_MX_1u -> Valve:SW_MX_1u
- ST-0: renamed from ST-0_0; value 7u -> 6.25u; footprint marbastlib-mx:STAB_MX_7u -> Valve:STAB_MX_6.25u
Connections:
- net col1: now also MX4-1.1 (COL); no longer MX4-1.2 (ROW)
- net col4: no longer MX4-5.1 (COL)
- net col5: now also MX4-5.1 (COL)
- net at MX4-5.2 (ROW): now also D59.2 (A)
- net at D57.2 (A): now also MX4-1.2 (ROW); no longer MX4-1.1 (COL)
Other:
- moved on the sheet: D59, MX4-0, MX4-1, MX4-5, ST-0
